File: ArduinoProjects/2015/_Done/122-Worlds_Tiniest_LED_Cube/eagle/TinyCube/TinyCube07_Hell_02.brd (EAGLE design)
At the start: 31.4 x 31.7 mm, 4 parts

Commit message: sync
Routing:
- net N$77: track 80.4 -> 0.00 mm, vias 2 -> 0
- net N$10: track 0.00 -> 49.5 mm, vias 0 -> 7
- net N$73: track 41.7 -> 21.9 mm, vias 1 -> 0
- net N$1: track 42.7 -> 28.1 mm
- net N$8: track 0.00 -> 1.08 mm
Changed lines of the file:
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@@
 <contactref element="JP2" pad="2"/>
 <contactref element="JP1" pad="2"/>
-<wire x1="2.54" y1="21.59" x2="6.35" y2="21.59" width="0.4064" layer="16"/>
-<wire x1="6.35" y1="21.59" x2="6.35" y2="20.828" width="0.4064" layer="16"/>
-<wire x1="6.35" y1="20.828" x2="10.668" y2="20.828" width="0.4064" layer="16"/>
-<wire x1="10.668" y1="20.828" x2="10.668" y2="15.748" width="0.4064" layer="16"/>
-<wire x1="11.43" y1="6.35" x2="10.668" y2="6.35" width="0.4064" layer="16"/>
-<wire x1="10.668" y1="6.35" x2="10.668" y2="15.748" width="0.4064" layer="16"/>
-<wire x1="10.668" y1="15.748" x2="16.51" y2="15.748" width="0.4064" layer="16"/>
-<wire x1="16.51" y1="16.51" x2="16.51" y2="15.748" width="0.4064" layer="16"/>
-<wire x1="16.51" y1="15.748" x2="23.368" y2="15.748" width="0.4064" layer="16"/>
-<wire x1="23.368" y1="15.748" x2="23.368" y2="11.43" width="0.4064" layer="16"/>
-<wire x1="23.368" y1="11.43" x2="24.13" y2="11.43" width="0.4064" layer="16"/>
-<wire x1="24.13" y1="11.43" x2="27.94" y2="21.59" width="0" layer="19" extent="1-16"/>
+<wire x1="12.7" y1="21.59" x2="12.7" y2="16.51" width="0.4064" layer="16"/>
+<wire x1="12.7" y1="16.51" x2="16.51" y2="12.7" width="0.4064" layer="16"/>
+<wire x1="16.51" y1="11.43" x2="16.51" y2="12.7" width="0.4064" layer="16"/>
+<wire x1="16.51" y1="12.7" x2="20.32" y2="16.51" width="0.4064" layer="16"/>
+<wire x1="20.32" y1="16.51" x2="22.86" y2="16.51" width="0.4064" layer="16"/>
+<wire x1="22.86" y1="16.51" x2="27.94" y2="21.59" width="0.4064" layer="16"/>
+<wire x1="12.7" y1="21.59" x2="11.43" y2="21.59" width="0.4064" layer="16"/>
+<wire x1="11.43" y1="21.59" x2="2.54" y2="21.59" width="0" layer="19" extent="1-16"/>
 </signal>
 <signal name="N$5">
@@
 <contactref element="JP2" pad="6"/>
 <contactref element="JP1" pad="6"/>
-<wire x1="2.54" y1="11.43" x2="27.94" y2="11.43" width="0" layer="19" extent="1-1"/>
+<wire x1="27.94" y1="11.43" x2="27.178" y2="10.668" width="0.4064" layer="16"/>
+<wire x1="27.178" y1="10.668" x2="2.54" y2="11.43" width="0" layer="19" extent="1-16"/>
 </signal>
 <signal name="N$9">
@@
 <contactref element="JP2" pad="8"/>
 <contactref element="JP1" pad="8"/>
-<wire x1="2.54" y1="6.35" x2="27.94" y2="6.35" width="0" layer="19" extent="1-1"/>
+<wire x1="27.94" y1="6.35" x2="25.146" y2="6.35" width="0.4064" layer="16"/>
+<wire x1="25.146" y1="6.35" x2="24.13" y2="5.334" width="0.4064" layer="16"/>
+<wire x1="24.13" y1="5.334" x2="22.606" y2="5.334" width="0.4064" layer="16"/>
+<wire x1="22.606" y1="5.334" x2="21.59" y2="6.35" width="0.4064" layer="16"/>
+<wire x1="21.59" y1="6.35" x2="22.352" y2="7.112" width="0.4064" layer="16"/>
+<wire x1="22.352" y1="7.112" x2="22.352" y2="15.24" width="0.4064" layer="16"/>
+<wire x1="21.59" y1="17.78" x2="20.32" y2="19.05" width="0.4064" layer="16"/>
+<wire x1="20.32" y1="19.05" x2="17.78" y2="21.59" width="0.4064" layer="16"/>
+<wire x1="17.78" y1="21.59" x2="15.24" y2="21.59" width="0.4064" layer="16"/>
+<wire x1="15.24" y1="21.59" x2="15.24" y2="16.51" width="0.4064" layer="16"/>
+<wire x1="12.7" y1="13.97" x2="11.43" y2="12.7" width="0.4064" layer="16"/>
+<wire x1="11.43" y1="12.7" x2="11.43" y2="11.43" width="0.4064" layer="16"/>
+<wire x1="10.16" y1="11.43" x2="8.89" y2="12.7" width="0" layer="19" extent="1-16"/>
+<wire x1="8.89" y1="12.7" x2="7.874" y2="12.7" width="0" layer="19" extent="1-16"/>
+<wire x1="7.874" y1="20.066" x2="6.35" y2="21.59" width="0" layer="19" extent="1-16"/>
+<via x="20.32" y="19.05" extent="1-16" drill="0.6" diameter="0.4064"/>
+<via x="22.352" y="15.24" extent="1-16" drill="0.6" diameter="0.4064"/>
+<via x="21.59" y="17.78" extent="1-16" drill="0.6" diameter="0.4064"/>
+<wire x1="21.59" y1="17.78" x2="22.352" y2="17.018" width="0.4064" layer="1"/>
+<wire x1="22.352" y1="17.018" x2="22.352" y2="15.24" width="0.4064" layer="1"/>
+<via x="15.24" y="16.51" extent="1-16" drill="0.6" diameter="0.4064"/>
+<via x="12.7" y="13.97" extent="1-16" drill="0.6" diameter="0.4064"/>
+<wire x1="12.7" y1="13.97" x2="15.24" y2="16.51" width="0.4064" layer="1"/>
+<wire x1="2.54" y1="6.35" x2="7.874" y2="12.7" width="0" layer="19" extent="16-16"/>
+<wire x1="7.874" y1="12.7" x2="7.874" y2="14.986" width="0" layer="19" extent="1-16"/>
+<wire x1="6.35" y1="16.51" x2="2.54" y2="6.35" width="0" layer="19" extent="1-16"/>
+<wire x1="7.874" y1="14.986" x2="6.35" y2="16.51" width="0" layer="19" extent="1-16"/>
+<wire x1="11.43" y1="11.43" x2="9.906" y2="11.43" width="0.4064" layer="16"/>
+<wire x1="9.906" y1="11.43" x2="9.906" y2="14.224" width="0.4064" layer="16"/>
+<wire x1="9.906" y1="14.224" x2="8.89" y2="15.24" width="0.4064" layer="16"/>
+<via x="8.89" y="15.24" extent="1-16" drill="0.6" diameter="0.4064"/>
+<wire x1="8.89" y1="15.24" x2="6.35" y2="17.78" width="0.4064" layer="1"/>
+<via x="6.35" y="17.78" extent="1-16" drill="0.6" diameter="0.4064"/>
+<wire x1="6.35" y1="17.78" x2="6.35" y2="16.51" width="0.4064" layer="16"/>
+<wire x1="6.35" y1="16.51" x2="2.54" y2="6.35" width="0" layer="19" extent="1-16"/>
 </signal>
 <signal name="N$13">
@@
 <contactref element="JP3" pad="1"/>
 <wire x1="6.35" y1="2.54" x2="6.35" y2="6.35" width="0.4064" layer="16"/>
-<wire x1="6.35" y1="6.35" x2="7.112" y2="6.35" width="0.4064" layer="16"/>
-<wire x1="7.112" y1="6.35" x2="7.112" y2="22.352" width="0.4064" layer="16"/>
-<wire x1="7.112" y1="22.352" x2="11.43" y2="22.352" width="0.4064" layer="16"/>
-<wire x1="11.43" y1="21.59" x2="11.43" y2="22.352" width="0.4064" layer="16"/>
-<wire x1="11.43" y1="22.352" x2="15.748" y2="22.352" width="0.4064" layer="16"/>
-<via x="15.748" y="22.352" extent="1-16" drill="0.6"/>
-<wire x1="15.748" y1="22.352" x2="15.748" y2="11.43" width="0.4064" layer="1"/>
-<wire x1="15.748" y1="11.43" x2="16.51" y2="11.43" width="0.4064" layer="1"/>
-<wire x1="16.51" y1="11.43" x2="6.35" y2="27.94" width="0" layer="19" extent="1-16"/>
+<wire x1="6.35" y1="6.35" x2="7.112" y2="7.112" width="0.4064" layer="16"/>
+<wire x1="7.112" y1="7.112" x2="7.112" y2="18.542" width="0.4064" layer="16"/>
+<wire x1="7.112" y1="18.542" x2="10.16" y2="21.59" width="0.4064" layer="16"/>
+<wire x1="10.16" y1="21.59" x2="11.43" y2="21.59" width="0.4064" layer="16"/>
+<wire x1="11.43" y1="21.59" x2="6.35" y2="27.94" width="0" layer="19" extent="1-16"/>
 </signal>
 <signal name="N$74">
@@
 <contactref element="JP4" pad="5"/>
 <contactref element="JP3" pad="5"/>
-<wire x1="16.51" y1="2.54" x2="16.51" y2="6.35" width="0.4064" layer="16"/>
-<wire x1="20.828" y1="21.59" x2="20.828" y2="11.43" width="0.4064" layer="16"/>
-<wire x1="20.828" y1="11.43" x2="16.51" y2="6.35" width="0.4064" layer="16"/>
-<wire x1="6.35" y1="11.43" x2="5.715" y2="12.065" width="0.4064" layer="16"/>
-<wire x1="5.715" y1="12.065" x2="0.762" y2="17.018" width="0.4064" layer="16"/>
-<wire x1="0.762" y1="17.018" x2="0.762" y2="30.734" width="0.4064" layer="16"/>
-<wire x1="0.762" y1="30.734" x2="16.51" y2="30.734" width="0.4064" layer="16"/>
-<wire x1="16.51" y1="6.35" x2="15.748" y2="7.112" width="0.4064" layer="16"/>
-<wire x1="15.748" y1="7.112" x2="12.7" y2="7.112" width="0.4064" layer="16"/>
-<wire x1="12.7" y1="7.112" x2="12.192" y2="7.112" width="0" layer="19" extent="1-16"/>
-<wire x1="10.16" y1="16.51" x2="5.715" y2="12.065" width="0.4064" layer="16"/>
-<wire x1="10.16" y1="16.51" x2="12.7" y2="16.51" width="0.4064" layer="16"/>
-<via x="12.7" y="16.51" extent="1-16" drill="0.6"/>
-<wire x1="12.7" y1="16.51" x2="12.7" y2="7.112" width="0.4064" layer="1"/>
-<via x="12.7" y="7.112" extent="1-16" drill="0.6"/>
-<wire x1="16.51" y1="30.734" x2="16.51" y2="27.94" width="0" layer="19" extent="16-16"/>
+<wire x1="16.51" y1="2.54" x2="16.51" y2="27.94" width="0" layer="19" extent="1-1"/>
 </signal>
 <signal name="N$78">
@@
 <signal name="N$82">
 </signal>
+<signal name="N$81">
+<via x="8.89" y="15.24" extent="1-16" drill="0.6" diameter="0.4064"/>
+</signal>
+<signal name="N$83">
+<via x="6.35" y="17.78" extent="1-16" drill="0.6" diameter="0.4064"/>
+</signal>
 </signals>
