File: ArduinoProjects/2015/_Done/122-Worlds_Tiniest_LED_Cube/eagle/TinyCube/TinyCube12 - Copy/TinyCube12a_Lib.brd (EAGLE design)
At the start: 25.4 x 20.3 mm, 18 parts

Commit message: cube backup
Parts:
- removed JP1, JP2: (no value), adafruit:1X08-BIG
- added U$17, U$18: TINY_HEADER_DEV, TinyHeader:TINY_HEADER_PKG
- moved U$5 6.35 mm to (5.08, 12.7)
- moved U$6 6.35 mm to (10.2, 12.7)
- moved U$7 6.35 mm to (15.2, 12.7)
- moved U$10 6.35 mm to (10.2, 7.62)
- moved U$11 6.35 mm to (15.2, 7.62)
- moved U$9 6.35 mm to (5.08, 7.62)
- moved U$13 6.35 mm to (5.08, 2.54)
- moved U$14 6.35 mm to (10.2, 2.54)
- moved U$15 6.35 mm to (15.2, 2.54)
- moved U$8 6.35 mm to (20.3, 12.7)
- moved U$1 6.35 mm to (5.08, 17.8)
- moved U$12 6.35 mm to (20.3, 7.62)
- moved U$16 6.35 mm to (20.3, 2.54)
- moved U$2 6.35 mm to (10.2, 17.8)
- moved U$3 6.35 mm to (15.2, 17.8)
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Connections:
- removed net N$1: JP1.3, U$12.+, U$15.+, U$2.+, U$5.+
- new net N$5: U$1.B, U$13.B, U$18.P$1, U$5.B, U$9.B
- new net N$6: U$12.B, U$16.B, U$18.P$7, U$4.B, U$8.B
- new net N$7: U$11.B, U$15.B, U$18.P$8, U$3.B, U$7.B
- new net N$8: U$10.B, U$14.B, U$18.P$2, U$2.B, U$6.B
- new net N$9: U$1.G, U$17.P$2, U$2.G, U$3.G, U$4.G
- net N$2: now also U$17.P$4, U$5.G, U$6.G, U$7.G, U$8.G; no longer JP1.7, U$10.+, U$13.+, U$4.+, U$7.+
- net N$3: now also U$10.G, U$11.G, U$12.G, U$17.P$6, U$9.G; no longer JP2.6, U$1.+, U$11.+, U$16.+, U$6.+
- net N$4: now also U$13.G, U$14.G, U$15.G, U$16.G, U$17.P$8; no longer JP2.3, U$14.+, U$3.+, U$8.+, U$9.+
Routing:
- net N$5: track 0.00 -> 37.2 mm
- net N$1: track 37.1 -> 0.00 mm, vias 1 -> 0
- net N$8: track 0.00 -> 32.1 mm
- net N$7: track 0.00 -> 27.1 mm
- net N$6: track 0.00 -> 22.0 mm
- net N$9: track 0.00 -> 20.9 mm
- net N$4: track 40.7 -> 20.9 mm, vias 1 -> 0
- net N$2: track 29.9 -> 20.9 mm
- net N$3: track 27.4 -> 20.9 mm
Other:
- board text added: "A"
- board text removed: "B"
