File: ArduinoProjects/2015/_Done/122-Worlds_Tiniest_LED_Cube/eagle/TinyCube/TinyCube12 - Copy/TinyCube12b_Lib.brd (EAGLE design)
At the start: 25.4 x 20.3 mm, 18 parts

Commit message: cube backup
Parts:
- removed JP1, JP2: (no value), adafruit:1X08-BIG
- added U$17, U$18: TINY_HEADER_DEV, TinyHeader:TINY_HEADER_PKG
Connections:
- net N$1: now also U$17.P$3; no longer JP1.3
- net N$2: now also U$17.P$7; no longer JP1.7
- net N$3: now also U$18.P$6; no longer JP2.6
- net N$4: now also U$18.P$3; no longer JP2.3
Other:
- outline, holes or cut-outs redrawn
Changed lines of the file:
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@@
 <setting verticaltext="up"/>
 </settings>
-<grid distance="10" unitdist="mil" unit="mil" style="lines" multiple="1" display="yes" altdistance="1" altunitdist="mil" altunit="mil"/>
+<grid distance="50" unitdist="mil" unit="mil" style="lines" multiple="1" display="yes" altdistance="1" altunitdist="mil" altunit="mil"/>
 <layers>
 <layer number="1" name="Top" color="4" fill="1" visible="yes" active="yes"/>
@@
 <layer number="21" name="tPlace" color="7" fill="1" visible="yes" active="yes"/>
 <layer number="22" name="bPlace" color="7" fill="1" visible="yes" active="yes"/>
-<layer number="23" name="tOrigins" color="15" fill="1" visible="no" active="yes"/>
-<layer number="24" name="bOrigins" color="15" fill="1" visible="no" active="yes"/>
-<layer number="25" name="tNames" color="7" fill="1" visible="no" active="yes"/>
-<layer number="26" name="bNames" color="7" fill="1" visible="no" active="yes"/>
+<layer number="23" name="tOrigins" color="15" fill="1" visible="yes" active="yes"/>
+<layer number="24" name="bOrigins" color="15" fill="1" visible="yes" active="yes"/>
+<layer number="25" name="tNames" color="7" fill="1" visible="yes" active="yes"/>
+<layer number="26" name="bNames" color="7" fill="1" visible="yes" active="yes"/>
 <layer number="27" name="tValues" color="7" fill="1" visible="no" active="yes"/>
 <layer number="28" name="bValues" color="7" fill="1" visible="yes" active="yes"/>
@@
 <board>
 <plain>
-<wire x1="3.81" y1="5.08" x2="29.2102" y2="5.08" width="0" layer="20"/>
+<wire x1="29.21" y1="5.08" x2="29.2102" y2="5.08" width="0" layer="20"/>
 <wire x1="29.2102" y1="5.08" x2="29.2102" y2="25.39" width="0" layer="20"/>
 <wire x1="29.2102" y1="25.39" x2="3.81" y2="25.39" width="0" layer="20"/>
@@
 <text x="6.604" y="24.13" size="0.4064" layer="25" align="center">A0</text>
 <text x="6.604" y="19.05" size="0.4064" layer="25" align="center">D11</text>
-<text x="5.842" y="17.78" size="0.4064" layer="25" align="center">D3</text>
-<text x="5.842" y="15.24" size="0.4064" layer="25" align="center">A2</text>
-<text x="5.842" y="12.7" size="0.4064" layer="25" align="center">D4</text>
-<text x="5.842" y="10.16" size="0.4064" layer="25" align="center">D13</text>
-<text x="5.842" y="7.62" size="0.4064" layer="25" align="center">D5</text>
-<text x="27.178" y="22.606" size="0.4064" layer="25" align="center">D8</text>
-<text x="27.178" y="25.146" size="0.4064" layer="25" align="center">D9</text>
-<text x="27.178" y="20.066" size="0.4064" layer="25" align="center">D12</text>
-<text x="27.178" y="17.526" size="0.4064" layer="25" align="center">A3</text>
-<text x="27.178" y="14.986" size="0.4064" layer="25" align="center">A1</text>
-<text x="27.178" y="12.446" size="0.4064" layer="25" align="center">D10</text>
-<text x="27.178" y="9.906" size="0.4064" layer="25" align="center">D6</text>
-<text x="27.178" y="7.366" size="0.4064" layer="25" align="center">D7</text>
+<text x="6.604" y="16.51" size="0.4064" layer="25" align="center">D3</text>
+<text x="6.604" y="13.97" size="0.4064" layer="25" align="center">A2</text>
+<text x="6.604" y="11.43" size="0.4064" layer="25" align="center">D4</text>
+<text x="6.604" y="8.89" size="0.4064" layer="25" align="center">D13</text>
+<text x="6.604" y="6.35" size="0.4064" layer="25" align="center">D5</text>
+<text x="26.67" y="21.59" size="0.4064" layer="25" align="center">D8</text>
+<text x="26.67" y="24.13" size="0.4064" layer="25" align="center">D9</text>
+<text x="26.67" y="19.05" size="0.4064" layer="25" align="center">D12</text>
+<text x="26.67" y="16.51" size="0.4064" layer="25" align="center">A3</text>
+<text x="26.67" y="13.97" size="0.4064" layer="25" align="center">A1</text>
+<text x="26.67" y="11.43" size="0.4064" layer="25" align="center">D10</text>
+<text x="26.67" y="8.89" size="0.4064" layer="25" align="center">D6</text>
+<text x="26.67" y="6.35" size="0.4064" layer="25" align="center">D7</text>
 <text x="10.922" y="19.304" size="1.778" layer="25">B</text>
+<wire x1="3.81" y1="25.4" x2="3.81" y2="5.08" width="0.4064" layer="20"/>
+<wire x1="3.81" y1="5.08" x2="29.21" y2="5.08" width="0.4064" layer="20"/>
+<wire x1="29.21" y1="5.08" x2="29.21" y2="25.146" width="0.4064" layer="20"/>
+<wire x1="3.81" y1="25.4" x2="29.21" y2="25.4" width="0.4064" layer="20"/>
+<wire x1="29.21" y1="25.4" x2="29.21" y2="25.146" width="0.4064" layer="20"/>
 </plain>
 <attributes>
@@
 </autorouter>
 <elements>
-<element name="JP1" library="adafruit" package="1X08-BIG" value="" x="5.08" y="15.24" smashed="yes" rot="R270">
-<attribute name="NAME" x="4.3688" y="25.4762" size="0.6096" layer="25" ratio="10" align="top-center" display="off"/>
-<attribute name="VALUE" x="1.905" y="25.4" size="1.27" layer="27" rot="R270"/>
-</element>
-<element name="JP2" library="adafruit" package="1X08-BIG" value="" x="27.94" y="15.24" smashed="yes" rot="R270">
-<attribute name="NAME" x="28.4988" y="25.4762" size="0.6096" layer="25" ratio="10" align="top-center" display="off"/>
-<attribute name="VALUE" x="24.765" y="25.4" size="1.27" layer="27" rot="R270"/>
-</element>
 <element name="U$1" library="PILLAR" package="10MIL" value="PILLAR" x="8.89" y="22.86"/>
 <element name="U$2" library="PILLAR" package="10MIL" value="PILLAR" x="13.97" y="22.86"/>
@@
 <element name="U$15" library="PILLAR" package="10MIL" value="PILLAR" x="19.05" y="7.62"/>
 <element name="U$16" library="PILLAR" package="10MIL" value="PILLAR" x="24.13" y="7.62"/>
+<element name="U$17" library="TinyHeader" package="TINY_HEADER_PKG" value="TINY_HEADER_DEV" x="5.08" y="24.13"/>
+<element name="U$18" library="TinyHeader" package="TINY_HEADER_PKG" value="TINY_HEADER_DEV" x="27.94" y="24.13"/>
 </elements>
 <signals>
 <signal name="N$2">
-<contactref element="JP1" pad="7"/>
 <contactref element="U$13" pad="+"/>
 <contactref element="U$10" pad="+"/>
 <contactref element="U$7" pad="+"/>
 <contactref element="U$4" pad="+"/>
-<wire x1="6.35" y1="7.62" x2="5.08" y2="8.89" width="0.4064" layer="16"/>
 <wire x1="10.16" y1="8.89" x2="10.16" y2="10.16" width="0.4064" layer="16"/>
 <wire x1="10.16" y1="10.16" x2="13.97" y2="13.97" width="0.4064" layer="16"/>
@@
 <wire x1="8.89" y1="8.89" x2="7.62" y2="7.62" width="0.4064" layer="16"/>
 <wire x1="7.62" y1="7.62" x2="6.35" y2="7.62" width="0.4064" layer="16"/>
+<contactref element="U$17" pad="P$7"/>
+<wire x1="5.08" y1="8.89" x2="6.35" y2="7.62" width="0.4064" layer="16"/>
 </signal>
 <signal name="N$4">
@@
 <wire x1="25.4" y1="20.32" x2="21.59" y2="24.13" width="0.4064" layer="1"/>
 <wire x1="21.59" y1="24.13" x2="20.32" y2="24.13" width="0.4064" layer="1"/>
-<contactref element="JP2" pad="3"/>
+<contactref element="U$18" pad="P$3"/>
 <wire x1="27.94" y1="19.05" x2="25.4" y2="19.05" width="0.4064" layer="1"/>
 </signal>
@@
 <contactref element="U$15" pad="+"/>
 <contactref element="U$12" pad="+"/>
-<contactref element="JP1" pad="3"/>
 <contactref element="U$5" pad="+"/>
 <contactref element="U$2" pad="+"/>
@@
 <wire x1="25.4" y1="15.24" x2="16.51" y2="24.13" width="0.4064" layer="1"/>
 <wire x1="16.51" y1="24.13" x2="15.24" y2="24.13" width="0.4064" layer="1"/>
-<wire x1="6.35" y1="17.78" x2="5.08" y2="19.05" width="0.4064" layer="16"/>
 <wire x1="7.62" y1="17.78" x2="6.35" y2="17.78" width="0.4064" layer="16"/>
 <wire x1="15.24" y1="24.13" x2="13.97" y2="24.13" width="0.4064" layer="16"/>
@@
 <wire x1="10.16" y1="19.05" x2="8.89" y2="19.05" width="0.4064" layer="16"/>
 <wire x1="8.89" y1="19.05" x2="7.62" y2="17.78" width="0.4064" layer="16"/>
+<contactref element="U$17" pad="P$3"/>
+<wire x1="5.08" y1="19.05" x2="6.35" y2="17.78" width="0.4064" layer="16"/>
 </signal>
 <signal name="N$3">
-<contactref element="JP2" pad="6"/>
 <contactref element="U$1" pad="+"/>
 <contactref element="U$6" pad="+"/>
@@
 <wire x1="15.24" y1="20.32" x2="11.43" y2="24.13" width="0.4064" layer="1"/>
 <wire x1="11.43" y1="24.13" x2="10.16" y2="24.13" width="0.4064" layer="1"/>
+<contactref element="U$18" pad="P$6"/>
 <wire x1="27.94" y1="11.43" x2="25.4" y2="8.89" width="0.4064" layer="1"/>
 </signal>
