File: ArduinoProjects/2015/_Done/122-Worlds_Tiniest_LED_Cube/eagle/TinyCube/TinyCube12 - Copy/TinyCube12c_Lib.brd (EAGLE design)
At the start: 25.4 x 20.3 mm, 18 parts

Commit message: cube backup
Parts:
- JP1, JP2: value (none) -> TINY_HEADER_DEV; device adafruit:1X08-BIG -> TinyHeader:TINY_HEADER_PKG
- moved U$5 6.35 mm to (5.08, 12.7)
- moved U$6 6.35 mm to (10.2, 12.7)
- moved U$7 6.35 mm to (15.2, 12.7)
- moved U$10 6.35 mm to (10.2, 7.62)
- moved U$11 6.35 mm to (15.2, 7.62)
- moved U$9 6.35 mm to (5.08, 7.62)
- moved U$13 6.35 mm to (5.08, 2.54)
- moved U$14 6.35 mm to (10.2, 2.54)
- moved U$15 6.35 mm to (15.2, 2.54)
- moved U$8 6.35 mm to (20.3, 12.7)
- moved U$1 6.35 mm to (5.08, 17.8)
- moved U$12 6.35 mm to (20.3, 7.62)
- moved U$16 6.35 mm to (20.3, 2.54)
- moved U$2 6.35 mm to (10.2, 17.8)
- moved U$3 6.35 mm to (15.2, 17.8)
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Connections:
- removed net N$4: JP2.3, U$14.+, U$3.+, U$8.+, U$9.+
- new net N$5: JP1.P$5, U$15.R, U$4.R, U$6.R, U$9.R
- net N$1: now also JP1.P$1, U$1.R, U$12.R, U$14.R, U$7.R; no longer JP1.3, U$12.+, U$15.+, U$2.+, U$5.+
- net N$2: now also JP2.P$4, U$11.R, U$13.R, U$2.R, U$8.R; no longer JP1.7, U$10.+, U$13.+, U$4.+, U$7.+
- net N$3: now also JP2.P$5, U$10.R, U$16.R, U$3.R, U$5.R; no longer JP2.6, U$1.+, U$11.+, U$16.+, U$6.+
Routing:
- net N$4: track 40.7 -> 0.00 mm, vias 1 -> 0
- net N$5: track 0.00 -> 35.7 mm
- net N$3: track 27.4 -> 40.4 mm
- net N$2: track 29.9 -> 39.3 mm
- net N$1: track 37.1 -> 35.7 mm, vias 1 -> 0
Other:
- board text added: "C"
- board text removed: "B"
